File: Kicad Files/KC65Clone.kicad_pcb (KiCad board)
At the start: 2 copper layers, 304.5 x 95 mm, 170 parts, among them J1 Conn_01x04, SW1 GRAVE, SW10 9, SW11 0, SW12 -, SW13 +, SW14 BSPC, SW15 DEL, SW16 TAB, SW17 Q, SW18 W, SW19 E, SW2 1, SW20 R, SW21 T, SW22 Y, SW23 U, SW24 I, SW25 O, SW26 P, SW27 [, SW28 ], SW29 SPLIT_BS, SW3 2, SW30 PGUP, SW31 CAPS, SW32 A, SW33 S, SW34 D, SW35 F, SW36 G, SW37 H, SW38 J, SW39 K, SW4 3, SW40 L, SW41 COLON, SW42 QUOTE, SW43 BSLS, SW44 ENTER, SW45 PGDN, SW46 LSFT, SW47 Z, SW48 X, SW49 C, SW5 4, SW50 V, SW51 B, SW52 N, SW53 M, SW54 COMMA, SW55 DOT, SW56 SLSH, SW57 RSFT, SW58 UP, SW59 END, SW6 5, SW60 LCTL, SW61 LGUI, SW62 LALT, SW63 6.25U SPC, SW64 RALT, SW65 RCTL, SW66 LEFT, SW67 DOWN, SW68 RIGHT, SW69 1.5U LCTL, SW7 6, SW70 1U LGUI, SW71 1.5U LALT, SW72 7U SPC, SW73 1.5U MO1, SW74 SPLIT_BSLS, SW75 STEPPED CAPS, SW8 7, SW9 8, U1 STM32F072C8Tx, U2 XC6206P332MR

Commit message: added holes
Parts:
- added ?: , , F.Cu at (122.7, 146.2)
- added ?: , , F.Cu at (160.8, 146.2)
- added ?: , , F.Cu at (256.1, 146.2)
- added ?: , , F.Cu at (294.2, 146.2)
- added C12: 4.7uF, Capacitor_SMD:C_0402_1005Metric, B.Cu at (83.5, 121.6)
- added REF**: OSHW-Symbol_8.9x8mm_SilkScreen, Symbol:OSHW-Symbol_8.9x8mm_SilkScreen, B.Cu at (176.0, 158.9)
- C6: value 100nF -> 1nF
- moved C1 11.9 mm to (92.8, 125.3), turned to 45 degrees
- moved C6 11.6 mm to (95.5, 114.4), turned to 135 degrees
- moved LED1 4.81 mm to (72.7, 124.0), turned to 0 degrees
- moved LED2 4.74 mm to (77.5, 124.0), turned to 180 degrees
- moved C2 2.63 mm to (96.2, 110.8)
- moved C7 1.66 mm to (96.6, 113.8)
- moved C11 1.26 mm to (88.4, 112.3)
- moved C4 1.24 mm to (88.4, 111.0)
- moved R2 1.09 mm to (79.9, 122.0)
- moved C5 0.87 mm to (82.5, 122.6)
- renumbered BOOT to SW76, RESET to SW77
Routing:
- net +3.3V: track 101.7 -> 104.6 mm
- net GND: track 59.6 -> 62.3 mm, vias 43 -> 45
- net Net-(LED1-A): track 7.07 -> 6.24 mm
Other:
- outline, holes or cut-outs redrawn
- board text added: "For No.2/65"
- board text added: "https://github.com/ThunderrGodd/KeyCult65ClonePCB"
- board text removed: "Kalam Cult No.2/65"

Commit message: Edited BackSplit
Parts:
- removed ? (x4): , 
- removed LED1, LED2: LED, LED_SMD:LED_1206_3216Metric_ReverseMount_Hole1.8x2.4mm
- removed R2: 470R, Resistor_SMD:R_0402_1005Metric
- removed the REF** at (325.2, 119.1)
- removed the REF** at (191.8, 157.2)
- removed the REF** at (82.3, 138.1)
- removed the REF** at (327.5, 81.0)
- removed the REF** at (203.7, 157.2)
- added H1: MountingHole, MountingHole:MountingHole_3.5mm, F.Cu at (122.7, 146.2)
- added H2: MountingHole, MountingHole:MountingHole_3.5mm, F.Cu at (160.8, 146.2)
- added H3: MountingHole, MountingHole:MountingHole_3.5mm, F.Cu at (256.1, 146.2)
- added H4: MountingHole, MountingHole:MountingHole_3.5mm, F.Cu at (294.2, 146.2)
- SW1, SW10, SW11, SW12, SW13, SW15, SW17, SW18, SW19, SW2, SW20, SW21, SW22, SW23, SW24, SW25, SW26, SW27, SW28, SW29, SW3, SW30, SW32, SW33, SW34, SW35, SW36, SW37, SW38, SW39, SW4, SW40, SW41, SW42, SW45, SW47, SW48, SW49, SW5, SW50, SW51, SW52, SW53, SW54, SW55, SW56, SW58, SW59, SW6, SW66, SW67, SW68, SW7, SW70, SW74, SW8, SW9: footprint PCM_Switch_Keyboard_Cherry_MX:SW_Cherry_MX_PCB_1.00u_valueprint -> CherryMX_PCB_NoSilk:CherryMX_1.00u_PCB
- SW14: footprint PCM_Switch_Keyboard_Cherry_MX:SW_Cherry_MX_PCB_2.00u_valueprint -> CherryMX_PCB_NoSilk:CherryMX_2.00u_PCB_StabWireBottom
- SW16, SW43, SW69, SW71, SW73: footprint PCM_Switch_Keyboard_Cherry_MX:SW_Cherry_MX_PCB_1.50u_valueprint -> CherryMX_PCB_NoSilk:CherryMX_1.50u_PCB
- SW31: footprint PCM_Switch_Keyboard_Cherry_MX:SW_Cherry_MX_PCB_1.75u_valueprint -> CherryMX_PCB_NoSilk:CherryMX_1.75u_PCB_LED
- SW44, SW46: footprint PCM_Switch_Keyboard_Cherry_MX:SW_Cherry_MX_PCB_2.25u_valueprint -> CherryMX_PCB_NoSilk:CherryMX_2.25u_PCB_StabWireBottom
- SW57: footprint PCM_Switch_Keyboard_Cherry_MX:SW_Cherry_MX_PCB_1.75u_valueprint -> CherryMX_PCB_NoSilk:CherryMX_1.75u_PCB
- SW60, SW61, SW62, SW64, SW65: footprint PCM_Switch_Keyboard_Cherry_MX:SW_Cherry_MX_PCB_1.25u_valueprint -> CherryMX_PCB_NoSilk:CherryMX_1.25u_PCB
- SW63: footprint PCM_Switch_Keyboard_Cherry_MX:SW_Cherry_MX_PCB_6.25u -> CherryMX_PCB_NoSilk:CherryMX_6.25u_PCB_StabWireTop
- SW72: footprint PCM_Switch_Keyboard_Cherry_MX:SW_Cherry_MX_PCB_7.00u -> CherryMX_PCB_NoSilk:CherryMX_7.00u_PCB_StabWireTop
- SW75: footprint PCM_Switch_Keyboard_Cherry_MX:SW_Cherry_MX_PCB_1.25u_valueprint -> CherryMX_PCB_NoSilk:CherryMX_1.25u_PCB_LED
- moved D64 1.06 mm to (111.5, 151.7)
- moved D75 1.01 mm to (328.2, 151.7)
- moved D71 1.00 mm to (254.4, 151.7)
- moved D68 0.98 mm to (183.0, 151.7)
- moved D76 0.97 mm to (347.2, 151.7)
- moved D74 0.90 mm to (309.1, 151.7)
- moved D63 0.88 mm to (87.8, 151.7)
- moved D62 0.83 mm to (83.8, 151.7)
- moved D73 0.82 mm to (275.9, 151.7)
- turned SW29 to 0 degrees
Connections:
- D32 pad 2: Net-(D32-A) -> ROW2
- SW31 pad 1: Net-(D32-A) -> ROW2
- SW75 pad 1: Net-(D32-A) -> ROW2
Routing:
- net ROW1: track 347.1 -> 298.7 mm
- net ROW2: track 363.3 -> 324.4 mm, vias 2 -> 4
- net GND: track 62.3 -> 42.6 mm, vias 45 -> 19
- net NRST: track 48.9 -> 34.4 mm
- net Net-(D32-A): track 11.2 -> 0.00 mm
- net Net-(D30-A): track 4.48 -> 14.0 mm
- net COL13: track 349.7 -> 356.4 mm
- net Net-(LED1-A): track 6.24 -> 0.00 mm
- net COL2: track 131.0 -> 126.5 mm
- net ROW0: track 326.4 -> 322.5 mm
- net COL12: track 336.2 -> 332.5 mm
- net Net-(D63-A): track 11.4 -> 7.88 mm
- net Net-(D64-A): track 11.3 -> 7.92 mm
- net COL1: track 125.4 -> 122.8 mm
- net +5V: track 23.0 -> 20.6 mm
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
Commit message: deleted readme.md
Parts:
- removed C11, C12: 4.7uF, Capacitor_SMD:C_0402_1005Metric
- removed C6: 1nF, Capacitor_SMD:C_0402_1005Metric
- removed C8: 100nF, Capacitor_SMD:C_0402_1005Metric
- removed D1: PRTR5V0U2X, Package_TO_SOT_SMD:SOT-143
- moved C2 2.82 mm to (94.5, 113.0)
- moved C7 1.86 mm to (95.4, 115.2)
- moved C5 1.53 mm to (83.6, 121.5)
- moved C4 1.28 mm to (88.4, 112.2)
Connections:
- D32 pad 2: ROW2 -> Net-(D32-A)
- SW31 pad 1: ROW2 -> Net-(D32-A)
- SW75 pad 1: ROW2 -> Net-(D32-A)
Routing:
- net +3.3V: track 103.6 -> 86.8 mm
- net GND: track 42.6 -> 29.8 mm, vias 19 -> 17
- net ROW2: track 324.4 -> 313.2 mm
- net Net-(D32-A): track 0.00 -> 10.8 mm
- net ROW4: track 310.2 -> 301.8 mm
- net +5V: track 20.6 -> 14.8 mm
- net D+: track 42.9 -> 40.2 mm
- net D-: track 43.5 -> 40.9 mm
- net CAPSLCK: track 19.9 -> 18.4 mm
- net NRST: track 34.4 -> 33.5 mm
- net COL2: track 126.5 -> 125.7 mm
- net COL13: track 356.4 -> 355.7 mm
Other:
- board text added: "1.25U"
- board text added: "1.5U"
- board text added: "1U"
- board text added: "LALT"
- board text added: "LCTRL"
- board text added: "LGUI"
- board text added: "RCTRL"
- board text removed: "1"
