File: Kicad Files/KC65Clone.kicad_pcb (KiCad board)
At the start: 2 copper layers, 304.5 x 95 mm, 163 parts, among them J1 Conn_01x04, SW1 GRAVE, SW10 9, SW11 0, SW12 -, SW13 +, SW14 BSPC, SW15 DEL, SW16 TAB, SW17 Q, SW18 W, SW19 E, SW2 1, SW20 R, SW21 T, SW22 Y, SW23 U, SW24 I, SW25 O, SW26 P, SW27 [, SW28 ], SW29 SPLIT_BS, SW3 2, SW30 PGUP, SW31 CAPS, SW32 A, SW33 S, SW34 D, SW35 F, SW36 G, SW37 H, SW38 J, SW39 K, SW4 3, SW40 L, SW41 COLON, SW42 QUOTE, SW43 BSLS, SW44 ENTER, SW45 PGDN, SW46 LSFT, SW47 Z, SW48 X, SW49 C, SW5 4, SW50 V, SW51 B, SW52 N, SW53 M, SW54 COMMA, SW55 DOT, SW56 SLSH, SW57 RSFT, SW58 UP, SW59 END, SW6 5, SW60 LCTL, SW61 LGUI, SW62 LALT, SW63 6.25U SPC, SW64 RALT, SW65 RCTL, SW66 LEFT, SW67 DOWN, SW68 RIGHT, SW69 1.5U LCTL, SW7 6, SW70 1U LGUI, SW71 1.5U LALT, SW72 7U SPC, SW73 1.5U MO1, SW74 SPLIT_BSLS, SW75 STEPPED CAPS, SW76 SKQGABE010, SW77 SKQGABE010, SW8 7, SW9 8, U1 STM32F072C8Tx, U2 XC6206P332MR

Commit message: updated pcb
Parts:
- D10, D11, D12, D13, D14, D15, D16, D17, D18, D19, D2, D20, D21, D22, D23, D24, D25, D26, D27, D28, D29, D3, D30, D31, D32, D33, D34, D35, D36, D37, D38, D39, D4, D40, D41, D42, D43, D44, D45, D46, D47, D49, D5, D50, D51, D52, D53, D54, D55, D56, D57, D58, D59, D6, D60, D61, D62, D63, D64, D68, D7, D71, D73, D74, D75, D76, D8, D9: footprint Diode_SMD:D_SOD-123 -> CherryMX_PCB_Value:D_SOD-123
- SW1, SW10, SW11, SW12, SW13, SW15, SW17, SW18, SW19, SW2, SW20, SW21, SW22, SW23, SW24, SW25, SW26, SW27, SW28, SW29, SW3, SW30, SW32, SW33, SW34, SW35, SW36, SW37, SW38, SW39, SW4, SW40, SW41, SW42, SW45, SW47, SW48, SW49, SW5, SW50, SW51, SW52, SW53, SW54, SW55, SW56, SW58, SW59, SW6, SW66, SW67, SW68, SW7, SW70, SW74, SW8, SW9: footprint CherryMX_PCB_NoSilk:CherryMX_1.00u_PCB -> CherryMX_PCB_Value:CherryMX_1.00u_PCB_silk
- moved D2 1.03 mm to (65.7, 85.4)
Routing:
- net ROW0: track 322.5 -> 324.1 mm
Other:
- board text added: "GND"
