File: Kicad Files/KC65Clone.kicad_sch (KiCad schematic)
At the start: 22 parts, among them J1 Conn_01x04, SW76 SKQGABE010, SW77 SKQGABE010, U1 STM32F072C8Tx, U2 XC6206P332MR

Commit message: added holes
Parts:
- added C12: 4.7uF, Capacitor_SMD:C_0402_1005Metric, symbol Device:C
- C6: value 100nF -> 1nF
Connections:
- net +3.3V: now also C12.1
- net GND: now also C12.2
Other:
- moved on the sheet: C1, C11, C2, C3, C4, C5, C6, C7, C8, D1, F1, J1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

Commit message: Edited BackSplit
Parts:
- removed LED1, LED2: LED, LED_SMD:LED_1206_3216Metric_ReverseMount_Hole1.8x2.4mm, symbol Device:LED
- removed R2: 470R, Resistor_SMD:R_0402_1005Metric, symbol Device:R_Small
- added H1, H2, H3, H4: MountingHole, MountingHole:MountingHole_3.5mm, symbol Mechanical:MountingHole

Commit message: deleted readme.md
Parts:
- removed C11, C12: 4.7uF, Capacitor_SMD:C_0402_1005Metric, symbol Device:C
- removed C6: 1nF, Capacitor_SMD:C_0402_1005Metric, symbol Device:C
- removed C8: 100nF, Capacitor_SMD:C_0402_1005Metric, symbol Device:C
- removed D1: PRTR5V0U2X, Package_TO_SOT_SMD:SOT-143, symbol Power_Protection:PRTR5V0U2X
